File: preamp.sch (KiCad schematic (older format))
At the start: 15 parts, among them J1 JACK_2P, U1 uA741CP

Commit message: perform simulation and analsysis add some images
Parts:
- added P1: OUT, ~, symbol CONN_2
- added P2: PWR, ~, symbol CONN_3
- J1: value JACK_2P -> MIC_IN
Connections:
- net +12V: now also P2.3 (P3)
- net +3.3VADC: now also P2.2 (PM)
- net GND: now also J1.3, P1.1 (P1), P2.1 (P1); no longer J1.1
- net Vout: now also P1.2 (PM)
- net at C1.1, R1.2: now also J1.1; no longer J1.3
Other:
- note added: "+PSPICE\n* \n*.op\n*.ac dec 10 1 50K\n*.plot ac vdb(1), vdb(8)\n\n.tran 0.1ms 3ms\n.plot tran v(1), v(8)\n"
- note added: "-PSPICE\n* \n.include components.cir"
- moved on the sheet: D1, D2, J1, R8
